Commit message: feat(T-017): integrate EtherCAT CSP Updown into 14-axis control
REQ-ECAT-001 REQ-ECAT-002 REQ-ECAT-004 REQ-ECAT-005 REQ-ECAT-006 REQ-ECAT-007

REQ-CAN-002 REQ-CAN-003 REQ-CAN-004 REQ-CAN-005 REQ-CAN-006 REQ-CAN-007

REQ-IF-001 REQ-IF-002 REQ-IF-004 REQ-IF-007

File: src/description/robot_description/urdf/robot.urdf.xacro (robot description, xacro)
@@ -603,5 +603,5 @@
     <child link="updown" />
     <axis xyz="0 0 1" />
-    <limit lower="0.0" upper="0.8" effort="0" velocity="0" />
+    <limit lower="0.0" upper="0.8" effort="0" velocity="0.3" />
   </joint>
   <joint name="front_sensor" type="fixed">

File: src/rt_control/robot_hw_canopen/urdf/canopen.ros2_control.xacro (robot description, xacro)
@@ -11,8 +11,4 @@
       <param name="can_interface_name">$(arg can_interface_name)</param>
     </hardware>
-    <joint name="updown">
-      <param name="node_id">1</param>
-      <param name="operation_mode">1</param>
-    </joint>
     <joint name="left_track_joint">
       <param name="node_id">2</param>

File: src/rt_control/robot_hw_ethercat/urdf/ecat.ros2_control.xacro (robot description, xacro)
@@ -34,4 +34,19 @@
     </joint>
   </xacro:macro>
+  <xacro:macro name="xmc_axis" params="joint_name ring_position profile">
+    <joint name="${joint_name}">
+      <command_interface name="position"/>
+      <command_interface name="control_word"/>
+      <state_interface name="position"/>
+      <state_interface name="status_word"/>
+      <ec_module name="${joint_name}_drive">
+        <plugin>ethercat_generic_plugins/EcCiA402Drive</plugin>
+        <param name="alias">0</param>
+        <param name="position">${ring_position}</param>
+        <param name="mode_of_operation">8</param>
+        <param name="slave_config">$(arg config_dir)/slaves/${profile}.yaml</param>
+      </ec_module>
+    </joint>
+  </xacro:macro>
   <ros2_control name="ecat_arms" type="system">
     <hardware>
@@ -55,4 +70,5 @@
     <xacro:zeroerr_axis joint_name="left_joint6" ring_position="12" profile="left_j6"/>
     <xacro:zeroerr_axis joint_name="turn" ring_position="14" profile="turn"/>
+    <xacro:xmc_axis joint_name="updown" ring_position="15" profile="xmc_updown_sw511"/>
     <sensor name="ethercat_domain">
       <state_interface name="process_data_age_ms"/>
@@ -76,4 +92,5 @@
     <sensor name="ethercat_slave_12"><state_interface name="al_state"/></sensor>
     <sensor name="ethercat_slave_14"><state_interface name="al_state"/></sensor>
+    <sensor name="ethercat_slave_15"><state_interface name="al_state"/></sensor>
   </ros2_control>
 </robot>

File: src/rt_control/rt_control_bringup/urdf/mock.ros2_control.xacro (robot description, xacro)
@@ -26,4 +26,5 @@
     <xacro:mock_ecat_axis joint_name="left_joint6"/>
     <xacro:mock_ecat_axis joint_name="turn"/>
+    <xacro:mock_ecat_axis joint_name="updown"/>
     <sensor name="ethercat_domain">
       <state_interface name="process_data_age_ms"><param name="initial_value">0.0</param></state_interface>
@@ -31,5 +32,5 @@
     <sensor name="ethercat_master">
       <state_interface name="link_up"><param name="initial_value">1.0</param></state_interface>
-      <state_interface name="slaves_responding"><param name="initial_value">15.0</param></state_interface>
+      <state_interface name="slaves_responding"><param name="initial_value">16.0</param></state_interface>
       <state_interface name="wc_error_count"><param name="initial_value">0.0</param></state_interface>
     </sensor>
@@ -47,4 +48,5 @@
     <sensor name="ethercat_slave_12"><state_interface name="al_state"><param name="initial_value">8.0</param></state_interface></sensor>
     <sensor name="ethercat_slave_14"><state_interface name="al_state"><param name="initial_value">8.0</param></state_interface></sensor>
+    <sensor name="ethercat_slave_15"><state_interface name="al_state"><param name="initial_value">8.0</param></state_interface></sensor>
   </ros2_control>
   <ros2_control name="canopen_mobile_axes" type="system">
@@ -52,12 +54,4 @@
       <plugin>mock_components/GenericSystem</plugin>
     </hardware>
-    <joint name="updown">
-      <command_interface name="position"/>
-      <command_interface name="tpdo/index"/>
-      <command_interface name="tpdo/subindex"/>
-      <command_interface name="tpdo/data"/>
-      <command_interface name="tpdo/ons"/>
-      <state_interface name="position"><param name="initial_value">0.0</param></state_interface>
-    </joint>
     <joint name="left_track_joint">
       <command_interface name="velocity"/>

Commit message: feat(T-020): publish navigation and vision TF tree
REQ: REQ-IF-003 REQ-MIG-003

Decision: AMB-017 BQ-123

File: src/description/robot_description/urdf/robot.urdf.xacro (robot description, xacro)
@@ -4,9 +4,10 @@
     Kinematics and meshes migrated from alfa_robot_description at
     8297e386b3fa8e8184820f7de5c91226c726bd94. Active-production overlays:
-    fixed pitch (BQ-062), bounded turn (BQ-060/BQ-061), and updown [0, 0.8] m (BQ-048).
+    base_footprint root (BQ-123), fixed pitch (BQ-062), bounded turn
+    (BQ-060/BQ-061), and updown [0, 0.8] m (BQ-048).
   -->
-  <link name="world"/>
-  <joint name="world_to_base" type="fixed">
-    <parent link="world"/>
+  <link name="base_footprint"/>
+  <joint name="base_footprint_to_base" type="fixed">
+    <parent link="base_footprint"/>
     <child link="base_link"/>
     <origin xyz="0 0 0.202094" rpy="0 0 0"/>

Commit message: fix(T-020): align perception sensor frames
REQ: REQ-IF-003 REQ-MIG-003

Decision: BQ-125

File: src/description/robot_description/urdf/robot.urdf.xacro (robot description, xacro)
@@ -497,5 +497,5 @@
     </collision>
   </link>
-  <link name="lidar_front">
+  <link name="lidar_front_mount">
     <inertial>
       <origin xyz="-6.42377262494165E-11 1.00857335138538E-05 0.00951653834947522" rpy="0 0 0" />
@@ -519,5 +519,9 @@
     </collision>
   </link>
-  <link name="lidar_rear">
+  <!-- Native installed MID360 frame; keep the CAD mesh on the mount link. -->
+  <link name="lidar_front"/>
+  <link name="livox_fused_frame"/>
+  <link name="top_sensor"/>
+  <link name="lidar_rear_mount">
     <inertial>
       <origin xyz="7.75510065591511E-05 1.02653775136408E-05 0.00951684895357141" rpy="0 0 0" />
@@ -541,4 +545,5 @@
     </collision>
   </link>
+  <link name="lidar_rear"/>
   <link name="cam_front">
     <inertial>
@@ -585,4 +590,6 @@
     </collision>
   </link>
+  <!-- REP-103 optical frame used by the top perception camera pipeline. -->
+  <link name="camera_top_color_optical_frame"/>
   <!-- Production phase: pitch is mechanically fixed at the source zero pose. -->
   <joint name="pitch" type="fixed">
@@ -612,24 +619,51 @@
     <axis xyz="0 0 0" />
   </joint>
-  <joint name="lidar_front" type="fixed">
+  <joint name="lidar_front_mount_joint" type="fixed">
     <origin xyz="0.16084 0 1.2155" rpy="0 0 0" />
     <parent link="turn" />
+    <child link="lidar_front_mount" />
+    <axis xyz="0 0 0" />
+  </joint>
+  <joint name="lidar_front_frame_joint" type="fixed">
+    <origin xyz="0 0 0" rpy="3.141592653589793 0 -1.570796326794897" />
+    <parent link="lidar_front_mount" />
     <child link="lidar_front" />
+  </joint>
+  <!-- Frame represented by dual_livox_fusion and FAST-LIO fused input. -->
+  <joint name="lidar_front_to_livox_fused_frame" type="fixed">
+    <origin xyz="0 0.175 0" rpy="3.141592653589793 0 0" />
+    <parent link="lidar_front" />
+    <child link="livox_fused_frame" />
+  </joint>
+  <!-- Conventional robot working frame: +X front, +Y left, +Z up. -->
+  <joint name="lidar_front_to_top_sensor" type="fixed">
+    <origin xyz="0 0 0" rpy="3.141592653589793 0 -1.570796326794897" />
+    <parent link="lidar_front" />
+    <child link="top_sensor" />
+  </joint>
+  <joint name="lidar_rear_mount_joint" type="fixed">
+    <origin xyz="-0.19316 0 1.2155" rpy="0 0 0" />
+    <parent link="turn" />
+    <child link="lidar_rear_mount" />
     <axis xyz="0 0 0" />
   </joint>
-  <joint name="lidar_rear" type="fixed">
-    <origin xyz="-0.193155597668545 0 1.2155009" rpy="0 0 0" />
-    <parent link="turn" />
+  <joint name="lidar_rear_frame_joint" type="fixed">
+    <origin xyz="0 0 0" rpy="3.141592653589793 0 -1.570796326794897" />
+    <parent link="lidar_rear_mount" />
     <child link="lidar_rear" />
-    <axis xyz="0 0 0" />
   </joint>
   <joint name="cam_front" type="fixed">
-    <origin xyz="0.224174685843815 0 1.28542950857142" rpy="0 0.261799387799146 0" />
+    <origin xyz="0.23667 0 1.2725" rpy="0 0.7854 0" />
     <parent link="turn" />
     <child link="cam_front" />
     <axis xyz="0 0 0" />
   </joint>
+  <joint name="cam_front_to_camera_top_color_optical_frame" type="fixed">
+    <origin xyz="0 0 0" rpy="-1.57079632679 0 -1.57079632679" />
+    <parent link="cam_front" />
+    <child link="camera_top_color_optical_frame" />
+  </joint>
   <joint name="cam_rear" type="fixed">
-    <origin xyz="-0.256485881180905 0 1.28542950857142" rpy="0 0.261799387799146 3.14159263525858" />
+    <origin xyz="-0.25649 0 1.2854" rpy="0 0.2618 3.1416" />
     <parent link="turn" />
     <child link="cam_rear" />

Commit message: fix(robot-model): offset base footprint by 15 cm

File: src/description/robot_description/urdf/robot.urdf.xacro (robot description, xacro)
@@ -11,5 +11,5 @@
     <parent link="base_footprint"/>
     <child link="base_link"/>
-    <origin xyz="0 0 0.202094" rpy="0 0 0"/>
+    <origin xyz="0.15 0 0.202094" rpy="0 0 0"/>
   </joint>
   <link name="base_link">

Commit message: feat(robot-model): add base-linked lidar_main TF [ELECTRI-106]
Add the user-supplied millimetre STL and preserve its base_link coordinates through the lidar_main fixed-frame geometry transform. Keep the public TF and asset contract documented and tested.

Refs: ELECTRI-106

File: src/description/robot_description/urdf/robot.urdf.xacro (robot description, xacro)
@@ -497,4 +497,27 @@
     </collision>
   </link>
+  <!-- The supplied STL is authored in base_link millimetres.  The inverse
+       visual/collision origin maps it into the lidar_main link frame. -->
+  <link name="lidar_main">
+    <visual>
+      <origin xyz="-0.270226881461 -0.133500000000 -0.296681769019"
+              rpy="0 -0.523598775598 0" />
+      <geometry>
+        <mesh filename="package://robot_description/meshes/current_robot/visual/lidar_main.STL"
+              scale="0.001 0.001 0.001" />
+      </geometry>
+      <material name="lidar_main_material">
+        <color rgba="0.752941176470588 0.752941176470588 0.752941176470588 1" />
+      </material>
+    </visual>
+    <collision>
+      <origin xyz="-0.270226881461 -0.133500000000 -0.296681769019"
+              rpy="0 -0.523598775598 0" />
+      <geometry>
+        <mesh filename="package://robot_description/meshes/current_robot/collision/lidar_main.STL"
+              scale="0.001 0.001 0.001" />
+      </geometry>
+    </collision>
+  </link>
   <link name="lidar_front_mount">
     <inertial>
@@ -619,4 +642,11 @@
     <axis xyz="0 0 0" />
   </joint>
+  <joint name="lidar_main_joint" type="fixed">
+    <origin xyz="0.382364228640 0.133500000000 0.121820508080"
+            rpy="0 0.523598775598 0" />
+    <parent link="base_link" />
+    <child link="lidar_main" />
+    <axis xyz="0 0 0" />
+  </joint>
   <joint name="lidar_front_mount_joint" type="fixed">
     <origin xyz="0.16084 0 1.2155" rpy="0 0 0" />
