Commit message: feat(rt-control): establish V3 integration baseline [ELECTRI-126]

File: src/description/robot_description/urdf/robot.urdf.xacro (robot description, xacro)
@@ -1,727 +1,36 @@
 <?xml version="1.0" encoding="UTF-8"?>
-<robot xmlns:xacro="http://wiki.ros.org/xacro" name="alfa_robot">
+<robot xmlns:xacro="http://wiki.ros.org/xacro" name="alfa_robot_v3">
   <!--
-    Kinematics and meshes migrated from alfa_robot_description at
-    8297e386b3fa8e8184820f7de5c91226c726bd94. Active-production overlays:
-    base_footprint root (BQ-123), fixed pitch (BQ-062), bounded turn
-    (BQ-060/BQ-061), and updown [0, 0.8] m (BQ-048).
+    ALFA V3.0.9 geometry and kinematics entrypoint.
+    end_effector:=suction (default) or end_effector:=gripper selects both tools.
+    This branch intentionally contains description assets only. Hardware
+    interfaces, MoveIt semantics, controller configuration and sensor
+    extrinsics belong to their owning packages and are not inferred here.
   -->
+  <xacro:arg name="end_effector" default="suction" />
+  <xacro:include filename="$(find robot_description)/urdf/robot_v3_0_9.xacro"/>
+  <xacro:include filename="$(find robot_description)/urdf/robot_v3_chassis.xacro"/>
+  <!-- Stable system-facing root frames. base_footprint is the ground reference;
+       base_link uses the measured V3 installation offset. -->
   <link name="base_footprint"/>
-  <joint name="base_footprint_to_base" type="fixed">
+  <joint name="base_footprint_to_base_link" type="fixed">
     <parent link="base_footprint"/>
     <child link="base_link"/>
-    <origin xyz="0.15 0 0.202094" rpy="0 0 0"/>
+    <origin xyz="0.195 0.015 0.400" rpy="0 0 0"/>
   </joint>
-  <link name="base_link">
-    <inertial>
-      <origin xyz="-0.230884916297589 -3.59403635404876E-05 0.0098300335923569" rpy="0 0 0" />
-      <mass value="452.331665683053" />
-      <inertia ixx="42.2528214496965" ixy="2.90433873714437E-05" ixz="5.298622447798" iyy="45.7349589120892" iyz="-7.53976926582118E-07" izz="73.6336356175808" />
-    </inertial>
-    <visual>
-      <origin xyz="0 0 0" rpy="0 0 0" />
-      <geometry>
-        <mesh filename="package://robot_description/meshes/current_robot/visual/base_link.STL" />
-      </geometry>
-      <material name="">
-        <color rgba="0.752941176470588 0.752941176470588 0.752941176470588 1" />
-      </material>
-    </visual>
-    <collision>
-      <origin xyz="0 0 0" rpy="0 0 0" />
-      <geometry>
-        <mesh filename="package://robot_description/meshes/current_robot/collision/base_link.STL" />
-      </geometry>
-    </collision>
-  </link>
-  <link name="pitch">
-    <inertial>
-      <origin xyz="-0.197223755735604 0.0545002751304142 0.0848583683408171" rpy="0 0 0" />
-      <mass value="31.6766900042973" />
-      <inertia ixx="0.518885879634885" ixy="2.02803902282039E-08" ixz="-0.0059164248689273" iyy="0.580169083875299" iyz="3.22538967435459E-07" izz="1.06295541093974" />
-    </inertial>
-    <visual>
-      <origin xyz="0 0 0" rpy="0 0 0" />
-      <geometry>
-        <mesh filename="package://robot_description/meshes/current_robot/visual/pitch.STL" />
-      </geometry>
-      <material name="">
-        <color rgba="0.752941176470588 0.752941176470588 0.752941176470588 1" />
-      </material>
-    </visual>
-    <collision>
-      <origin xyz="0 0 0" rpy="0 0 0" />
-      <geometry>
-        <mesh filename="package://robot_description/meshes/current_robot/collision/pitch.STL" />
-      </geometry>
-    </collision>
-  </link>
-  <link name="turn">
-    <inertial>
-      <origin xyz="-0.0095811094528917 -7.73859721447945E-06 1.06018839944043" rpy="0 0 0" />
-      <mass value="53.4681885650186" />
-      <inertia ixx="7.9404350019494" ixy="5.99860879539091E-06" ixz="0.185339515626497" iyy="8.17240800709107" iyz="-8.94803411825732E-06" izz="0.75519185821394" />
-    </inertial>
-    <visual>
-      <origin xyz="0 0 0" rpy="0 0 0" />
-      <geometry>
-        <mesh filename="package://robot_description/meshes/current_robot/visual/turn.STL" />
-      </geometry>
-      <material name="">
-        <color rgba="0.752941176470588 0.752941176470588 0.752941176470588 1" />
-      </material>
-    </visual>
-    <collision>
-      <origin xyz="0 0 0" rpy="0 0 0" />
-      <geometry>
-        <mesh filename="package://robot_description/meshes/current_robot/collision/turn.STL" />
-      </geometry>
-    </collision>
-  </link>
-  <link name="updown">
-    <inertial>
-      <origin xyz="0.0637333774739139 -2.92604740437241E-09 0.104211014753682" rpy="0 0 0" />
-      <mass value="24.4167257440598" />
-      <inertia ixx="1.07967195604977" ixy="-1.55435028640832E-08" ixz="-0.00582099906204058" iyy="0.231957862842844" iyz="9.04966113481007E-11" izz="1.26737556353379" />
-    </inertial>
-    <visual>
-      <origin xyz="0 0 0" rpy="0 0 0" />
-      <geometry>
-        <mesh filename="package://robot_description/meshes/current_robot/visual/updown.STL" />
-      </geometry>
-      <material name="">
-        <color rgba="0.752941176470588 0.752941176470588 0.752941176470588 1" />
-      </material>
-    </visual>
-    <collision>
-      <origin xyz="0 0 0" rpy="0 0 0" />
-      <geometry>
-        <mesh filename="package://robot_description/meshes/current_robot/collision/updown.STL" />
-      </geometry>
-    </collision>
-  </link>
-  <!-- ========== LEFT ARM mapped to project names ========== -->
-  <link name="left_arm_base">
-    <inertial>
-      <origin xyz="0 0 0" rpy="0 0 0"/>
-      <mass value="0.001"/>
-      <inertia ixx="1e-6" ixy="0" ixz="0" iyy="1e-6" iyz="0" izz="1e-6"/>
-    </inertial>
-  </link>
-  <joint name="left_arm_mount" type="fixed">
-    <parent link="updown"/>
-    <child link="left_arm_base"/>
-    <origin xyz="0.095 0.26 0.2" rpy="0 0 0"/>
+  <link name="base_link"/>
+  <!-- CAD chassis root is 45.584858 mm above its plate bottom. The wheels
+       extend 320 mm below that bottom; preserve the existing chassis XY center. -->
+  <joint name="base_to_chassis" type="fixed">
+    <parent link="base_link"/>
+    <child link="chassis_base"/>
+    <origin xyz="-0.19 0 -0.034415142" rpy="0 0 0"/>
   </joint>
-  <link name="left_joint1">
-    <inertial>
-      <origin xyz="1.98132632578396E-05 0.0024729821757461 0.0580356323599247" rpy="0 0 0" />
-      <mass value="2.53849365971092" />
-      <inertia ixx="0.00565316591359222" ixy="1.39299660382164E-06" ixz="-2.78630772107311E-06" iyy="0.00554455173094155" iyz="-7.06906283259906E-05" izz="0.00447417412424819" />
-    </inertial>
-    <visual>
-      <origin xyz="0 0 0" rpy="0 0 0" />
-      <geometry>
-        <mesh filename="package://robot_description/meshes/current_robot/visual/leftjoint1.STL" />
-      </geometry>
-      <material name="">
-        <color rgba="0.752941176470588 0.752941176470588 0.752941176470588 1" />
-      </material>
-    </visual>
-    <collision>
-      <origin xyz="0 0 0" rpy="0 0 0" />
-      <geometry>
-        <mesh filename="package://robot_description/meshes/current_robot/collision/leftjoint1.STL" />
-      </geometry>
-    </collision>
-  </link>
-  <joint name="left_joint1" type="revolute">
-    <origin xyz="0 0 0" rpy="0 0 0" />
-    <parent link="left_arm_base" />
-    <child link="left_joint1" />
-    <axis xyz="0 0 1" />
-    <limit lower="-2.35619449" upper="2.35619449" effort="120" velocity="1.2" />
+  <joint name="base_to_model" type="fixed">
+    <parent link="base_link"/>
+    <child link="model_base"/>
+    <origin
+      xyz="-0.190000017371 6.50500004219e-09 0.662499964909"
+      rpy="1.5707963 0 1.57079632679"/>
   </joint>
-  <link name="left_joint2">
-    <inertial>
-      <origin xyz="-3.91993260073775E-09 -0.198242241905537 0.0685963634370466" rpy="0 0 0" />
-      <mass value="13.5734229269593" />
-      <inertia ixx="0.347009291103137" ixy="1.79329294469621E-12" ixz="2.19848376530362E-12" iyy="0.0505989087942828" iyz="4.33552705015945E-12" izz="0.367314390536816" />
-    </inertial>
-    <visual>
-      <origin xyz="0 0 0" rpy="0 0 0" />
-      <geometry>
-        <mesh filename="package://robot_description/meshes/current_robot/visual/leftjoint2.STL" />
-      </geometry>
-      <material name="">
-        <color rgba="0.752941176470588 0.752941176470588 0.752941176470588 1" />
-      </material>
-    </visual>
-    <collision>
-      <origin xyz="0 0 0" rpy="0 0 0" />
-      <geometry>
-        <mesh filename="package://robot_description/meshes/current_robot/collision/leftjoint2.STL" />
-      </geometry>
-    </collision>
-  </link>
-  <joint name="left_joint2" type="revolute">
-    <origin xyz="0 0.0825 0.058" rpy="-1.5708 0 0" />
-    <parent link="left_joint1" />
-    <child link="left_joint2" />
-    <axis xyz="0 0 1" />
-    <limit lower="-1.57079633" upper="1.57079633" effort="120" velocity="1.2" />
-  </joint>
-  <link name="left_joint3">
-    <inertial>
-      <origin xyz="2.86018788653308E-08 -0.174995964436896 -0.0214654505916678" rpy="0 0 0" />
-      <mass value="5.46918956371602" />
-      <inertia ixx="0.102635037762556" ixy="1.82331494669218E-08" ixz="3.03709958770067E-09" iyy="0.0138225294833702" iyz="4.39575520960004E-05" izz="0.114289616262011" />
-    </inertial>
-    <visual>
-      <origin xyz="0 0 0" rpy="0 0 0" />
-      <geometry>
-        <mesh filename="package://robot_description/meshes/current_robot/visual/leftjoint3.STL" />
-      </geometry>
-      <material name="">
-        <color rgba="0.752941176470588 0.752941176470588 0.752941176470588 1" />
-      </material>
-    </visual>
-    <collision>
-      <origin xyz="0 0 0" rpy="0 0 0" />
-      <geometry>
-        <mesh filename="package://robot_description/meshes/current_robot/collision/leftjoint3.STL" />
-      </geometry>
-    </collision>
-  </link>
-  <joint name="left_joint3" type="revolute">
-    <origin xyz="0 -0.4 0.008" rpy="0 0 0" />
-    <parent link="left_joint2" />
-    <child link="left_joint3" />
-    <axis xyz="0 0 1" />
-    <limit lower="-3.14159265" upper="3.14159265" effort="100" velocity="1.2" />
-  </joint>
-  <link name="left_joint4">
-    <inertial>
-      <origin xyz="1.79301766545237E-05 0.0022398818670486 0.0513862987308302" rpy="0 0 0" />
-      <mass value="2.80270206383319" />
-      <inertia ixx="0.00725799360950605" ixy="1.39369533421895E-06" ixz="-2.78625386086696E-06" iyy="0.00714937209205323" iyz="-7.06885588698108E-05" izz="0.00491856957816283" />
-    </inertial>
-    <visual>
-      <origin xyz="0 0 0" rpy="0 0 0" />
-      <geometry>
-        <mesh filename="package://robot_description/meshes/current_robot/visual/leftjoint4.STL" />
-      </geometry>
-      <material name="">
-        <color rgba="0.752941176470588 0.752941176470588 0.752941176470588 1" />
-      </material>
-    </visual>
-    <collision>
-      <origin xyz="0 0 0" rpy="0 0 0" />
-      <geometry>
-        <mesh filename="package://robot_description/meshes/current_robot/collision/leftjoint4.STL" />
-      </geometry>
-    </collision>
-  </link>
-  <joint name="left_joint4" type="revolute">
-    <origin xyz="0 -0.34 0.036" rpy="0 0 3.14159265" />
-    <parent link="left_joint3" />
-    <child link="left_joint4" />
-    <axis xyz="0 0 1" />
-    <limit lower="-3.14159265" upper="3.14159265" effort="60" velocity="1.5" />
-  </joint>
-  <link name="left_joint5">
-    <inertial>
-      <origin xyz="0.00232761885815957 1.86282466611079E-05 -0.0541835932362768" rpy="0 0 0" />
-      <mass value="2.69701788961683" />
-      <inertia ixx="0.00644984661938273" ixy="1.39391456329041E-06" ixz="7.06885192213968E-05" iyy="0.00655846677979015" iyz="2.78593765647904E-06" izz="0.00474081002137964" />
-    </inertial>
-    <visual>
-      <origin xyz="0 0 0" rpy="0 0 0" />
-      <geometry>
-        <mesh filename="package://robot_description/meshes/current_robot/visual/leftjoint5.STL" />
-      </geometry>
-      <material name="">
-        <color rgba="0.752941176470588 0.752941176470588 0.752941176470588 1" />
-      </material>
-    </visual>
-    <collision>
-      <origin xyz="0 0 0" rpy="0 0 0" />
-      <geometry>
-        <mesh filename="package://robot_description/meshes/current_robot/collision/leftjoint5.STL" />
-      </geometry>
-    </collision>
-  </link>
-  <joint name="left_joint5" type="revolute">
-    <origin xyz="0 0.076 0.058" rpy="-1.5708 0 3.14159265" />
-    <parent link="left_joint4" />
-    <child link="left_joint5" />
-    <axis xyz="0 0 1" />
-    <limit lower="-3.14159265" upper="3.14159265" effort="60" velocity="1.5" />
-  </joint>
-  <link name="left_joint6">
-    <inertial>
-      <origin xyz="0.000656912040293556 0.000831354479587647 0.143020209405828" rpy="0 0 0" />
-      <mass value="9.66858880038425" />
-      <inertia ixx="0.0956031747008674" ixy="2.07680535688619E-07" ixz="-3.59179174235467E-07" iyy="0.073686444653942" iyz="-1.65114179069294E-07" izz="0.104451818743786" />
-    </inertial>
-    <visual>
-      <origin xyz="0 0 0" rpy="0 0 0" />
-      <geometry>
-        <mesh filename="package://robot_description/meshes/current_robot/visual/leftjoint6.STL" />
-      </geometry>
-      <material name="">
-        <color rgba="0.752941176470588 0.752941176470588 0.752941176470588 1" />
-      </material>
-    </visual>
-    <collision>
-      <origin xyz="0 0 0" rpy="0 0 0" />
-      <geometry>
-        <mesh filename="package://robot_description/meshes/current_robot/collision/leftjoint6.STL" />
-      </geometry>
-    </collision>
-  </link>
-  <joint name="left_joint6" type="revolute">
-    <origin xyz="0.0825 0 -0.058" rpy="0 1.5708 0" />
-    <parent link="left_joint5" />
-    <child link="left_joint6" />
-    <axis xyz="0 0 1" />
-    <limit lower="-3.14159265" upper="3.14159265" effort="40" velocity="1.5" />
-  </joint>
-  <!-- ========== RIGHT ARM mapped to project names ========== -->
-  <link name="right_arm_base">
-    <inertial>
-      <origin xyz="0 0 0" rpy="0 0 0"/>
-      <mass value="0.001"/>
-      <inertia ixx="1e-6" ixy="0" ixz="0" iyy="1e-6" iyz="0" izz="1e-6"/>
-    </inertial>
-  </link>
-  <joint name="right_arm_mount" type="fixed">
-    <parent link="updown"/>
-    <child link="right_arm_base"/>
-    <origin xyz="0.095 -0.26 0.2" rpy="0 0 0"/>
-  </joint>
-  <link name="right_joint1">
-    <inertial>
-      <origin xyz="-1.97935614578704E-05 -0.00247298310211252 0.0580356306667533" rpy="0 0 0" />
-      <mass value="2.53849328920251" />
-      <inertia ixx="0.00565316574735245" ixy="1.3934599584903E-06" ixz="2.78607721450309E-06" iyy="0.00554455177196281" iyz="7.06907347564618E-05" izz="0.00447417409155335" />
-    </inertial>
-    <visual>
-      <origin xyz="0 0 0" rpy="0 0 0" />
-      <geometry>
-        <mesh filename="package://robot_description/meshes/current_robot/visual/rightjoint1.STL" />
-      </geometry>
-      <material name="">
-        <color rgba="0.752941176470588 0.752941176470588 0.752941176470588 1" />
-      </material>
-    </visual>
-    <collision>
-      <origin xyz="0 0 0" rpy="0 0 0" />
-      <geometry>
-        <mesh filename="package://robot_description/meshes/current_robot/collision/rightjoint1.STL" />
-      </geometry>
-    </collision>
-  </link>
-  <joint name="right_joint1" type="revolute">
-    <origin xyz="0 0 0" rpy="0 0 0" />
-    <parent link="right_arm_base" />
-    <child link="right_joint1" />
-    <axis xyz="0 0 1" />
-    <limit lower="-2.35619449" upper="2.35619449" effort="120" velocity="1.2" />
-  </joint>
-  <link name="right_joint2">
-    <inertial>
-      <origin xyz="-3.93094157224994E-09 -0.198242241906288 -0.0685963669555529" rpy="0 0 0" />
-      <mass value="13.573422926924" />
-      <inertia ixx="0.347009291103142" ixy="-1.77065393597298E-12" ixz="2.09998863566369E-12" iyy="0.0505989087942401" iyz="-4.27592541614651E-12" izz="0.367314390536786" />
-    </inertial>
-    <visual>
-      <origin xyz="0 0 0" rpy="0 0 0" />
-      <geometry>
-        <mesh filename="package://robot_description/meshes/current_robot/visual/rightjoint2.STL" />
-      </geometry>
-      <material name="">
-        <color rgba="0.752941176470588 0.752941176470588 0.752941176470588 1" />
-      </material>
-    </visual>
-    <collision>
-      <origin xyz="0 0 0" rpy="0 0 0" />
-      <geometry>
-        <mesh filename="package://robot_description/meshes/current_robot/collision/rightjoint2.STL" />
-      </geometry>
-    </collision>
-  </link>
-  <joint name="right_joint2" type="revolute">
-    <origin xyz="0 -0.0825 0.058" rpy="-1.5708 0 0" />
-    <parent link="right_joint1" />
-    <child link="right_joint2" />
-    <axis xyz="0 0 1" />
-    <limit lower="-1.57079633" upper="1.57079633" effort="120" velocity="1.2" />
-  </joint>
-  <link name="right_joint3">
-    <inertial>
-      <origin xyz="-2.19745741603106E-08 -0.174995898002215 0.0214654414595061" rpy="0 0 0" />
-      <mass value="5.4691844498613" />
-      <inertia ixx="0.102634928752236" ixy="5.65369033783247E-09" ixz="4.23974883669152E-09" iyy="0.0138225144033142" iyz="-4.3961229805213E-05" izz="0.114289495613127" />
-    </inertial>
-    <visual>
-      <origin xyz="0 0 0" rpy="0 0 0" />
-      <geometry>
-        <mesh filename="package://robot_description/meshes/current_robot/visual/rightjoint3.STL" />
-      </geometry>
-      <material name="">
-        <color rgba="0.752941176470588 0.752941176470588 0.752941176470588 1" />
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