Commit message: feat(rt-control): migrate V3.1.1 robot model [ELECTRI-136]

File: src/description/robot_description/urdf/robot.urdf (robot description, URDF)
Before this commit: robot alfa_robot_v3, 35 links, 34 joints
Links:
- removed link left_joint1
- removed link left_joint2
- removed link left_joint3
- removed link left_joint4
- removed link left_joint5
- removed link left_joint6
- removed link left_joint7
- removed link right_joint1
- removed link right_joint2
- removed link right_joint3
- removed link right_joint4
- removed link right_joint5
- removed link right_joint6
- removed link right_joint7
- added link chest_camera, mass 0.137417570647; collision mesh filename=package://robot_description/meshes/head_chest_camera/part_0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 scale=0.001 0.001 0.001; visual mesh filename=package://robot_description/meshes/head_chest_camera/part_0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 scale=0.001 0.001 0.001
- added link left_link1, mass 3.4800785; collision mesh filename=package://robot_description/meshes/robot_v3_1_1/part_022_so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 scale=0.001 0.001 0.001; visual mesh filename=package://robot_description/meshes/robot_v3_1_1/part_022_so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 scale=0.001 0.001 0.001
- added link left_link2, mass 4.2029403; collision mesh filename=package://robot_description/meshes/robot_v3_1_1/part_023_so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 scale=0.001 0.001 0.001; visual mesh filename=package://robot_description/meshes/robot_v3_1_1/part_023_so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 scale=0.001 0.001 0.001
- added link left_link3, mass 3.6348934; collision mesh filename=package://robot_description/meshes/robot_v3_1_1/part_024_so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 scale=0.001 0.001 0.001; visual mesh filename=package://robot_description/meshes/robot_v3_1_1/part_024_so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 scale=0.001 0.001 0.001
- added link left_link4, mass 3.5816422; collision mesh filename=package://robot_description/meshes/robot_v3_1_1/part_025_so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 scale=0.001 0.001 0.001; visual mesh filename=package://robot_description/meshes/robot_v3_1_1/part_025_so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 scale=0.001 0.001 0.001
- added link left_link5, mass 2.5714853; collision mesh filename=package://robot_description/meshes/robot_v3_1_1/part_026_so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 scale=0.001 0.001 0.001; visual mesh filename=package://robot_description/meshes/robot_v3_1_1/part_026_so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 scale=0.001 0.001 0.001
- added link left_link6, mass 0.4671032; collision mesh filename=package://robot_description/meshes/robot_v3_1_1/part_027_so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 scale=0.001 0.001 0.001; visual mesh filename=package://robot_description/meshes/robot_v3_1_1/part_027_so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 scale=0.001 0.001 0.001
- added link left_link7, mass 2.618; collision mesh filename=package://robot_description/meshes/robot_v3/suction_collisi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 scale=0.001 0.001 0.001; visual mesh filename=package://robot_description/meshes/robot_v3/suction_visual.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 scale=0.001 0.001 0.001
- added link right_link1, mass 3.4800784; collision mesh filename=package://robot_description/meshes/robot_v3_1_1/part_031_so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 scale=0.001 0.001 0.001; visual mesh filename=package://robot_description/meshes/robot_v3_1_1/part_031_so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 scale=0.001 0.001 0.001
- added link right_link2, mass 4.20294; collision mesh filename=package://robot_description/meshes/robot_v3_1_1/part_032_so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 scale=0.001 0.001 0.001; visual mesh filename=package://robot_description/meshes/robot_v3_1_1/part_032_so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 scale=0.001 0.001 0.001
- added link right_link3, mass 3.6348933; collision mesh filename=package://robot_description/meshes/robot_v3_1_1/part_033_so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 scale=0.001 0.001 0.001; visual mesh filename=package://robot_description/meshes/robot_v3_1_1/part_033_so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 scale=0.001 0.001 0.001
- added link right_link4, mass 3.5816414; collision mesh filename=package://robot_description/meshes/robot_v3_1_1/part_034_so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 scale=0.001 0.001 0.001; visual mesh filename=package://robot_description/meshes/robot_v3_1_1/part_034_so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 scale=0.001 0.001 0.001
- added link right_link5, mass 2.5714852; collision mesh filename=package://robot_description/meshes/robot_v3_1_1/part_035_so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 scale=0.001 0.001 0.001; visual mesh filename=package://robot_description/meshes/robot_v3_1_1/part_035_so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 scale=0.001 0.001 0.001
- added link right_link6, mass 0.4671031; collision mesh filename=package://robot_description/meshes/robot_v3_1_1/part_036_so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 scale=0.001 0.001 0.001; visual mesh filename=package://robot_description/meshes/robot_v3_1_1/part_036_so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 scale=0.001 0.001 0.001
- added link right_link7, mass 2.618; collision mesh filename=package://robot_description/meshes/robot_v3/suction_collisi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 scale=0.001 0.001 0.001; visual mesh filename=package://robot_description/meshes/robot_v3/suction_visual.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 scale=0.001 0.001 0.001
- link head: mass 0.19975472 -> 1.00116361294; geometry collision mesh filename=package://robot_description/meshes/head_chest_camera/part_0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 scale=0.001 0.001 0.001; collision mesh filename=package://robot_description/meshes/head_chest_camera/part_0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 scale=0.001 0.001 0.001
- link head_mount: mass 0.11917571 -> None; geometry 
- link head_yaw: mass 0.15476448 -> 0.07210205; geometry collision mesh filename=package://robot_description/meshes/head_chest_camera/part_0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 scale=0.001 0.001 0.001; visual mesh filename=package://robot_description/meshes/head_chest_camera/part_0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 scale=0.001 0.001 0.001
Joints:
- added joint chest_camera_fixed: type fixed, parent arm_carriage, child chest_camera, origin xyz=0.366 -3.92e-09 1.11530000583 rpy=0 0 0
- joint base_footprint_to_base_link: origin xyz=0.195 0.015 0.400 rpy=0 0 0 -> xyz=0.190000002779484 -0.0000442724271391554 0.40000250599116 rpy=0 0 0
- joint head_joint: origin xyz=0 0 0.005 rpy=0 0 0 -> xyz=0 0 0 rpy=0 0 0
- joint head_mount_fixed: origin xyz=0.226 0 1.3806412 rpy=0 0 0 -> xyz=0.267 0 1.4228 rpy=0 0 1.57079632679
- joint head_pitch_joint: origin xyz=0.04 0.005 0.05 rpy=-1.5707963 0 0 -> xyz=0.01393364 0.022 0.044 rpy=0 -1.5707963 0
- joint left_arm_mount: origin xyz=0 0 0 rpy=0 0 0 -> xyz=0 0 -0.0142 rpy=0 0 1.57079632679
- joint left_joint1: child left_joint1 -> left_link1; limit lower=-3.14159265 upper=3.14159265 effort=10 velocity=5 -> lower=-3.14159265 upper=3.14159265 effort=647 velocity=1.309; origin xyz=0.181 0.35372443 1.309511 rpy=-2.22044604925e-16 -1.3089969 -1.57079628038 -> xyz=0.32201385 -0.181 1.3500054 rpy=0 -1.3089969 3.1415927
- joint left_joint2: child left_joint2 -> left_link2; limit lower=-1.8325957145940461 upper=1.8325957145940461 effort=10 velocity=5 -> lower=-1.8325957145940461 upper=1.8325957145940461 effort=647 velocity=1.309; origin xyz=0.039999999 0 0.1272 rpy=0 -1.5707963 0 -> xyz=0.039999999 0 0.1512 rpy=0 -1.5707963 -3.1415927; parent left_joint1 -> left_link1
- joint left_joint3: child left_joint3 -> left_link3; limit lower=-3.14159265 upper=3.14159265 effort=10 velocity=5 -> lower=-3.14159265 upper=3.14159265 effort=484 velocity=1.309; origin xyz=0.1795 0 0.040000001 rpy=0 1.5707963 0 -> xyz=0.1795 0 -0.040000001 rpy=0 -1.5707963 3.1415927; parent left_joint2 -> left_link2
- joint left_joint4: child left_joint4 -> left_link4; limit lower=-2.53072742 upper=2.53072742 effort=10 velocity=5 -> lower=-2.53072742 upper=2.53072742 effort=459 velocity=1.749; origin xyz=-1.2261866e-09 0.07 0.3265 rpy=1.5707963 -1.3089969 -3.1415927 -> xyz=-1.2261866e-09 -0.068 0.3265 rpy=1.5707963 -1.3089969 -3.1415927; parent left_joint3 -> left_link3
- joint left_joint5: child left_joint5 -> left_link5; limit lower=-3.14159265 upper=3.14159265 effort=10 velocity=5 -> lower=-3.14159265 upper=3.14159265 effort=217 velocity=2.618; origin xyz=0.22457775 0.060175428 -0.07 rpy=-1.5707963 0 -1.30899695 -> xyz=0.22457775 0.060175428 0.068 rpy=1.5707963 0 1.8325957; parent left_joint4 -> left_link4
- joint left_joint6: child left_joint6 -> left_link6; limit lower=-1.91986218 upper=1.91986218 effort=10 velocity=5 -> lower=-1.91986218 upper=1.91986218 effort=107 velocity=3.142; origin xyz=0.076499999 0 0.2405 rpy=0 -1.5707963 -3.1415927 -> xyz=0.061499999 0 0.2415 rpy=0 -1.5707963 -3.1415927; parent left_joint5 -> left_link5
- joint left_joint7: child left_joint7 -> left_link7; limit lower=-3.14159265 upper=3.14159265 effort=10 velocity=5 -> lower=-3.14159265 upper=3.14159265 effort=36 velocity=3.142; origin xyz=0.1025 0 -0.0765 rpy=0 1.5707963 0 -> xyz=0.0993 0 -0.0615 rpy=0 -1.5707963 3.1415927; parent left_joint6 -> left_link6
- joint left_tool0_fixed: parent left_joint7 -> left_link7
- joint right_arm_mount: origin xyz=0 0 0 rpy=0 0 0 -> xyz=0 0 -0.0142 rpy=0 0 1.57079632679
- joint right_joint1: child right_joint1 -> right_link1; limit lower=-3.14159265 upper=3.14159265 effort=10 velocity=5 -> lower=-3.14159265 upper=3.14159265 effort=647 velocity=1.309; origin xyz=0.181 -0.33054221 1.3032993 rpy=3.33066907388e-16 -1.3089969 1.57079632679 -> xyz=-0.33054221 -0.181 1.3500054 rpy=0 -1.3089969 0
- joint right_joint2: child right_joint2 -> right_link2; limit lower=-1.8325957145940461 upper=1.8325957145940461 effort=10 velocity=5 -> lower=-1.8325957145940461 upper=1.8325957145940461 effort=647 velocity=1.309; origin xyz=0.039999999 0 0.1512 rpy=0 1.5707963 -3.1415927 -> xyz=0.039999999 0 0.1512 rpy=0 1.5707963 0; parent right_joint1 -> right_link1
- joint right_joint3: child right_joint3 -> right_link3; limit lower=-3.14159265 upper=3.14159265 effort=10 velocity=5 -> lower=-3.14159265 upper=3.14159265 effort=484 velocity=1.309; origin xyz=-0.1795 0 0.040000001 rpy=0 1.5707963 3.1415927 -> xyz=-0.1795 0 -0.040000001 rpy=0 -1.5707963 0; parent right_joint2 -> right_link2
- joint right_joint4: child right_joint4 -> right_link4; limit lower=-2.53072742 upper=2.53072742 effort=10 velocity=5 -> lower=-2.53072742 upper=2.53072742 effort=459 velocity=1.749; origin xyz=-1.2287747e-09 -0.068 0.3265 rpy=1.5707963 1.3089969 0 -> xyz=-1.2287747e-09 0.068 0.3265 rpy=1.5707963 1.3089969 0; parent right_joint3 -> right_link3
- joint right_joint5: child right_joint5 -> right_link5; limit lower=-3.14159265 upper=3.14159265 effort=10 velocity=5 -> lower=-3.14159265 upper=3.14159265 effort=217 velocity=2.618; origin xyz=-0.22457775 0.060175428 -0.068 rpy=-1.5707963 0 1.3089969 -> xyz=-0.22457775 0.060175428 0.068 rpy=-1.5707963 0 1.3089969; parent right_joint4 -> right_link4
- joint right_joint6: child right_joint6 -> right_link6; limit lower=-1.91986218 upper=1.91986218 effort=10 velocity=5 -> lower=-1.91986218 upper=1.91986218 effort=107 velocity=3.142; origin xyz=0.061499999 0 0.2405 rpy=0 1.5707963 0 -> xyz=0.061499999 0 0.2415 rpy=0 1.5707963 0; parent right_joint5 -> right_link5
- joint right_joint7: child right_joint7 -> right_link7; limit lower=-3.14159265 upper=3.14159265 effort=10 velocity=5 -> lower=-3.14159265 upper=3.14159265 effort=36 velocity=3.142; origin xyz=-0.1025 0 -0.0615 rpy=0 -1.5707963 0 -> xyz=-0.0993 0 -0.0615 rpy=0 -1.5707963 0; parent right_joint6 -> right_link6
- joint right_tool0_fixed: parent right_joint7 -> right_link7
- joint updown: limit lower=-0.5 upper=0.5 effort=1000 velocity=0.15 -> lower=-1 upper=0 effort=10 velocity=5; origin xyz=-6.505e-09 -1.14829997 0.19 rpy=-1.57079632679 -1.5707963 0 -> xyz=-6.50744829443e-09 -0.64829997 0.19 rpy=-1.57079632679 -1.5707963 0

File: src/description/robot_description/urdf/robot.urdf.xacro (robot description, xacro)
@@ -2,5 +2,5 @@
 <robot xmlns:xacro="http://wiki.ros.org/xacro" name="alfa_robot_v3">
   <!--
-    ALFA V3.0.9 geometry and kinematics entrypoint.
+    ALFA V3.1.1 arm/updown integration entrypoint.
     end_effector:=suction (default) or end_effector:=gripper selects both tools.
     This branch intentionally contains description assets only. Hardware
@@ -9,5 +9,5 @@
   -->
   <xacro:arg name="end_effector" default="suction" />
-  <xacro:include filename="$(find robot_description)/urdf/robot_v3_0_9.xacro"/>
+  <xacro:include filename="$(find robot_description)/urdf/robot_v3_1_1.xacro"/>
   <xacro:include filename="$(find robot_description)/urdf/robot_v3_chassis.xacro"/>
   <!-- Stable system-facing root frames. base_footprint is the ground reference;
@@ -17,5 +17,5 @@
     <parent link="base_footprint"/>
     <child link="base_link"/>
-    <origin xyz="0.195 0.015 0.400" rpy="0 0 0"/>
+    <origin xyz="0.190000002779484 -0.0000442724271391554 0.40000250599116" rpy="0 0 0"/>
   </joint>
   <link name="base_link"/>
