Commit message: feat(rt-control): migrate V3.1.1 robot model [ELECTRI-136]

File: src/description/robot_description/urdf/robot_v3_1_1.xacro (robot description, xacro)
@@ -1,8 +1,9 @@
 <?xml version="1.0" encoding="UTF-8"?>
 <!--
-  机身与机械臂沿用已校核的 V3.0.9 坐标、零位和限位。
-  末端支持双夹爪和双吸盘；上游 left/right 按 ROS 物理侧交换命名。
+  V3.1.1 双臂运动链集成到 Kkozia 模块化整机。
+  底盘、主动悬挂、双轴头部、夹爪/吸盘和 Tool0 保持目标分支定义。
+  Updown 保持同一 1m 实体行程，重标为 -1m 最低、0m 最高。
 -->
-<robot xmlns:xacro="http://wiki.ros.org/xacro" name="robot_v3_0_9_model">
+<robot xmlns:xacro="http://wiki.ros.org/xacro" name="robot_v3_1_1_hybrid_model">
   <xacro:arg name="end_effector" default="suction" />
   <xacro:include filename="$(find robot_description)/urdf/robot_v3_end_effectors.xacro" />
@@ -293,266 +294,230 @@
     </collision>
   </link>
-  <link name="right_joint1">
-    <inertial>
-      <origin xyz="0.026713084 -0.00035041447 0.12770383" rpy="0 0 0" />
-      <mass value="3.480078" />
-      <inertia ixx="0.019990668" iyy="0.023084509" izz="0.018380902" ixy="-1.7697786e-05" ixz="-0.00075602927" iyz="-8.1890221e-05" />
-    </inertial>
-    <visual>
-      <material name="robot_v3_gray">
-        <color rgba="0.82 0.82 0.82 1" />
-      </material>
-      <origin xyz="-0.3012366 0.261 -0.65601757" rpy="1.5707963 1.3089969 0" />
-      <geometry>
-        <mesh filename="package://robot_description/meshes/robot_v3/part_030_solid_030.stl" scale="0.001 0.001 0.001" />
-      </geometry>
-    </visual>
-    <collision>
-      <origin xyz="-0.3012366 0.261 -0.65601757" rpy="1.5707963 1.3089969 0" />
-      <geometry>
-        <mesh filename="package://robot_description/meshes/robot_v3/part_030_solid_030.stl" scale="0.001 0.001 0.001" />
-      </geometry>
-    </collision>
-  </link>
-  <link name="right_joint2">
-    <inertial>
-      <origin xyz="-0.16099656 2.2026045e-08 0.040000128" rpy="0 0 0" />
-      <mass value="4.3865152" />
-      <inertia ixx="0.015567361" iyy="0.017259138" izz="0.0233165" ixy="-9.7889543e-09" ixz="-5.7104315e-08" iyz="-1.0317529e-08" />
-    </inertial>
-    <visual>
-      <material name="robot_v3_gray">
-        <color rgba="0.82 0.82 0.82 1" />
-      </material>
-      <origin xyz="0.80721757 -0.261 0.34123659" rpy="-1.5707963 0.26179939 0" />
-      <geometry>
-        <mesh filename="package://robot_description/meshes/robot_v3/part_031_solid_031.stl" scale="0.001 0.001 0.001" />
-      </geometry>
-    </visual>
-    <collision>
-      <origin xyz="0.80721757 -0.261 0.34123659" rpy="-1.5707963 0.26179939 0" />
-      <geometry>
-        <mesh filename="package://robot_description/meshes/robot_v3/part_031_solid_031.stl" scale="0.001 0.001 0.001" />
-      </geometry>
-    </collision>
-  </link>
-  <link name="right_joint3">
-    <inertial>
-      <origin xyz="-5.6955242e-08 9.0900244e-10 0.23006341" rpy="0 0 0" />
+  <link name="right_link1">
+    <inertial>
+      <origin xyz="0.026713078 -0.00035041598 0.12770383" rpy="0 0 0" />
+      <mass value="3.4800784" />
+      <inertia ixx="0.019990671" iyy="0.023084514" izz="0.018380907" ixy="-1.7698217e-05" ixz="-0.00075603007" iyz="-8.1890443e-05" />
+    </inertial>
+    <visual>
+      <origin xyz="-0.34635123 0.261 -0.668106" rpy="1.5707963 1.3089969 0" />
+      <geometry>
+        <mesh filename="package://robot_description/meshes/robot_v3_1_1/part_031_solid_031.stl" scale="0.001 0.001 0.001" />
+      </geometry>
+    </visual>
+    <collision>
+      <origin xyz="-0.34635123 0.261 -0.668106" rpy="1.5707963 1.3089969 0" />
+      <geometry>
+        <mesh filename="package://robot_description/meshes/robot_v3_1_1/part_031_solid_031.stl" scale="0.001 0.001 0.001" />
+      </geometry>
+    </collision>
+  </link>
+  <link name="right_link2">
+    <inertial>
+      <origin xyz="-0.16472334 -1.1230144e-08 -0.040000126" rpy="0 0 0" />
+      <mass value="4.20294" />
+      <inertia ixx="0.014698616" iyy="0.015742815" izz="0.021103613" ixy="6.0405033e-09" ixz="5.5773205e-08" iyz="2.0954468e-08" />
+    </inertial>
+    <visual>
+      <origin xyz="0.819306 0.261 -0.38635123" rpy="1.5707963 -0.26179939 0" />
+      <geometry>
+        <mesh filename="package://robot_description/meshes/robot_v3_1_1/part_032_solid_032.stl" scale="0.001 0.001 0.001" />
+      </geometry>
+    </visual>
+    <collision>
+      <origin xyz="0.819306 0.261 -0.38635123" rpy="1.5707963 -0.26179939 0" />
+      <geometry>
+        <mesh filename="package://robot_description/meshes/robot_v3_1_1/part_032_solid_032.stl" scale="0.001 0.001 0.001" />
+      </geometry>
+    </collision>
+  </link>
+  <link name="right_link3">
+    <inertial>
+      <origin xyz="-5.896457e-08 9.5061022e-10 0.23006341" rpy="0 0 0" />
+      <mass value="3.6348933" />
+      <inertia ixx="0.039501207" iyy="0.037988453" izz="0.011543294" ixy="-2.7986338e-10" ixz="-1.0220005e-08" iyz="2.5352711e-09" />
+    </inertial>
+    <visual>
+      <origin xyz="-0.34635123 0.261 -0.998806" rpy="1.5707963 1.3089969 0" />
+      <geometry>
+        <mesh filename="package://robot_description/meshes/robot_v3_1_1/part_033_solid_033.stl" scale="0.001 0.001 0.001" />
+      </geometry>
+    </visual>
+    <collision>
+      <origin xyz="-0.34635123 0.261 -0.998806" rpy="1.5707963 1.3089969 0" />
+      <geometry>
+        <mesh filename="package://robot_description/meshes/robot_v3_1_1/part_033_solid_033.stl" scale="0.001 0.001 0.001" />
+      </geometry>
+    </collision>
+  </link>
+  <link name="right_link4">
+    <inertial>
+      <origin xyz="-0.12628065 0.0338368 0.067995266" rpy="0 0 0" />
+      <mass value="3.5816414" />
+      <inertia ixx="0.016515852" iyy="0.034995692" izz="0.029719473" ixy="0.0053346708" ixz="2.262619e-06" iyz="-6.0604321e-07" />
+    </inertial>
+    <visual>
+      <origin xyz="1.190505 -0.67756403 -0.193" rpy="0 0 0" />
+      <geometry>
+        <mesh filename="package://robot_description/meshes/robot_v3_1_1/part_034_solid_034.stl" scale="0.001 0.001 0.001" />
+      </geometry>
+    </visual>
+    <collision>
+      <origin xyz="1.190505 -0.67756403 -0.193" rpy="0 0 0" />
+      <geometry>
+        <mesh filename="package://robot_description/meshes/robot_v3_1_1/part_034_solid_034.stl" scale="0.001 0.001 0.001" />
+      </geometry>
+    </collision>
+  </link>
+  <link name="right_link5">
+    <inertial>
+      <origin xyz="-0.026166805 0 0.12943329" rpy="0 0 0" />
+      <mass value="2.5714852" />
+      <inertia ixx="0.0133841" iyy="0.016999468" izz="0.0092322376" ixy="-4.8880228e-11" ixz="-0.00036895645" iyz="-3.280144e-11" />
+    </inertial>
+    <visual>
+      <origin xyz="-0.34635123 0.261 -1.557806" rpy="1.5707963 1.3089969 0" />
+      <geometry>
+        <mesh filename="package://robot_description/meshes/robot_v3_1_1/part_035_solid_035.stl" scale="0.001 0.001 0.001" />
+      </geometry>
+    </visual>
+    <collision>
+      <origin xyz="-0.34635123 0.261 -1.557806" rpy="1.5707963 1.3089969 0" />
+      <geometry>
+        <mesh filename="package://robot_description/meshes/robot_v3_1_1/part_035_solid_035.stl" scale="0.001 0.001 0.001" />
+      </geometry>
+    </collision>
+  </link>
+  <link name="right_link6">
+    <inertial>
+      <origin xyz="-0.05437806 0 -0.061500007" rpy="0 0 0" />
+      <mass value="0.4671031" />
+      <inertia ixx="0.00042456776" iyy="0.00052425348" izz="0.00053281307" ixy="1.7956352e-12" ixz="-9.302396e-11" iyz="2.7467158e-12" />
+    </inertial>
+    <visual>
+      <origin xyz="1.799306 0.261 -0.40785123" rpy="1.5707963 -0.26179939 0" />
+      <geometry>
+        <mesh filename="package://robot_description/meshes/robot_v3_1_1/part_036_solid_036.stl" scale="0.001 0.001 0.001" />
+      </geometry>
+    </visual>
+    <collision>
+      <origin xyz="1.799306 0.261 -0.40785123" rpy="1.5707963 -0.26179939 0" />
+      <geometry>
+        <mesh filename="package://robot_description/meshes/robot_v3_1_1/part_036_solid_036.stl" scale="0.001 0.001 0.001" />
+      </geometry>
+    </collision>
+  </link>
+  <xacro:call macro="v3_$(arg end_effector)" side="right" />
+  <link name="left_link1">
+    <inertial>
+      <origin xyz="0.026713079 -0.00035041871 0.12770383" rpy="0 0 0" />
+      <mass value="3.4800785" />
+      <inertia ixx="0.019990672" iyy="0.023084515" izz="0.018380907" ixy="-1.7697964e-05" ixz="-0.00075602927" iyz="-8.1890411e-05" />
+    </inertial>
+    <visual>
+      <origin xyz="-0.46510803 -0.261 -0.22489961" rpy="1.5707963 -1.3089969 -3.1415927" />
+      <geometry>
+        <mesh filename="package://robot_description/meshes/robot_v3_1_1/part_022_solid_022.stl" scale="0.001 0.001 0.001" />
+      </geometry>
+    </visual>
+    <collision>
+      <origin xyz="-0.46510803 -0.261 -0.22489961" rpy="1.5707963 -1.3089969 -3.1415927" />
+      <geometry>
+        <mesh filename="package://robot_description/meshes/robot_v3_1_1/part_022_solid_022.stl" scale="0.001 0.001 0.001" />
+      </geometry>
+    </collision>
+  </link>
+  <link name="left_link2">
+    <inertial>
+      <origin xyz="0.16472335 1.2730856e-08 -0.040000127" rpy="0 0 0" />
+      <mass value="4.2029403" />
+      <inertia ixx="0.014698617" iyy="0.015742817" izz="0.021103615" ixy="5.4991019e-09" ixz="-5.5614112e-08" iyz="-2.0916153e-08" />
+    </inertial>
+    <visual>
+      <origin xyz="-0.37609961 0.261 -0.50510803" rpy="1.5707963 0.26179939 0" />
+      <geometry>
+        <mesh filename="package://robot_description/meshes/robot_v3_1_1/part_023_solid_023.stl" scale="0.001 0.001 0.001" />
+      </geometry>
+    </visual>
+    <collision>
+      <origin xyz="-0.37609961 0.261 -0.50510803" rpy="1.5707963 0.26179939 0" />
+      <geometry>
+        <mesh filename="package://robot_description/meshes/robot_v3_1_1/part_023_solid_023.stl" scale="0.001 0.001 0.001" />
+      </geometry>
+    </collision>
+  </link>
+  <link name="left_link3">
+    <inertial>
+      <origin xyz="-5.9080015e-08 2.5764869e-09 0.23006341" rpy="0 0 0" />
       <mass value="3.6348934" />
-      <inertia ixx="0.039501205" iyy="0.037988452" izz="0.011543295" ixy="-2.7434165e-10" ixz="-1.1101938e-08" iyz="2.5256667e-09" />
-    </inertial>
-    <visual>
-      <material name="robot_v3_gray">
-        <color rgba="0.82 0.82 0.82 1" />
-      </material>
-      <origin xyz="-0.30123659 0.261 -0.98671757" rpy="1.5707963 1.3089969 0" />
-      <geometry>
-        <mesh filename="package://robot_description/meshes/robot_v3/part_032_solid_032.stl" scale="0.001 0.001 0.001" />
-      </geometry>
-    </visual>
-    <collision>
-      <origin xyz="-0.30123659 0.261 -0.98671757" rpy="1.5707963 1.3089969 0" />
-      <geometry>
-        <mesh filename="package://robot_description/meshes/robot_v3/part_032_solid_032.stl" scale="0.001 0.001 0.001" />
-      </geometry>
-    </collision>
-  </link>
-  <link name="right_joint4">
-    <inertial>
-      <origin xyz="-0.12628065 0.033836795 -0.068004734" rpy="0 0 0" />
-      <mass value="3.5816415" />
-      <inertia ixx="0.016515852" iyy="0.034995692" izz="0.029719473" ixy="0.0053346702" ixz="2.2625524e-06" iyz="-6.0611007e-07" />
-    </inertial>
-    <visual>
-      <material name="robot_v3_gray">
-        <color rgba="0.82 0.82 0.82 1" />
-      </material>
-      <origin xyz="1.190505 -0.63085793 -0.329" rpy="0 0 0" />
-      <geometry>
-        <mesh filename="package://robot_description/meshes/robot_v3/part_033_solid_033.stl" scale="0.001 0.001 0.001" />
-      </geometry>
-    </visual>
-    <collision>
-      <origin xyz="1.190505 -0.63085793 -0.329" rpy="0 0 0" />
-      <geometry>
-        <mesh filename="package://robot_description/meshes/robot_v3/part_033_solid_033.stl" scale="0.001 0.001 0.001" />
-      </geometry>
-    </collision>
-  </link>
-  <link name="right_joint5">
-    <inertial>
-      <origin xyz="-0.026243466 5.8789419e-10 0.12878599" rpy="0 0 0" />
-      <mass value="2.5639754" />
-      <inertia ixx="0.013271124" iyy="0.016881335" izz="0.0092195991" ixy="-5.8734845e-11" ixz="-0.00039269041" iyz="-7.9121614e-11" />
-    </inertial>
-    <visual>
-      <material name="robot_v3_gray">
-        <color rgba="0.82 0.82 0.82 1" />
-      </material>
-      <origin xyz="-0.30123659 0.261 -1.5457176" rpy="1.5707963 1.3089969 0" />
-      <geometry>
-        <mesh filename="package://robot_description/meshes/robot_v3/part_034_solid_034.stl" scale="0.001 0.001 0.001" />
-      </geometry>
-    </visual>
-    <collision>
-      <origin xyz="-0.30123659 0.261 -1.5457176" rpy="1.5707963 1.3089969 0" />
-      <geometry>
-        <mesh filename="package://robot_description/meshes/robot_v3/part_034_solid_034.stl" scale="0.001 0.001 0.001" />
-      </geometry>
-    </collision>
-  </link>
-  <link name="right_joint6">
-    <inertial>
-      <origin xyz="-0.055950548 -3.659148e-10 -0.061500003" rpy="0 0 0" />
-      <mass value="0.48344395" />
-      <inertia ixx="0.00043921862" iyy="0.00056576363" izz="0.00057432331" ixy="-5.52059e-13" ixz="6.1707526e-11" iyz="-6.0033184e-13" />
-    </inertial>
-    <visual>
-      <material name="robot_v3_gray">
-        <color rgba="0.82 0.82 0.82 1" />
-      </material>
-      <origin xyz="1.7862176 0.261 -0.36273659" rpy="1.5707963 -0.26179939 0" />
-      <geometry>
-        <mesh filename="package://robot_description/meshes/robot_v3/part_035_solid_035.stl" scale="0.001 0.001 0.001" />
-      </geometry>
-    </visual>
-    <collision>
-      <origin xyz="1.7862176 0.261 -0.36273659" rpy="1.5707963 -0.26179939 0" />
-      <geometry>
-        <mesh filename="package://robot_description/meshes/robot_v3/part_035_solid_035.stl" scale="0.001 0.001 0.001" />
-      </geometry>
-    </collision>
-  </link>
-  <xacro:call macro="v3_$(arg end_effector)" side="right" />
-  <link name="left_joint1">
-    <inertial>
-      <origin xyz="0.026713085 -0.00035041698 0.10370383" rpy="0 0 0" />
-      <mass value="3.480078" />
-      <inertia ixx="0.019990668" iyy="0.023084509" izz="0.018380903" ixy="-1.7697502e-05" ixz="-0.00075602846" iyz="-8.1890176e-05" />
-    </inertial>
-    <visual>
-      <material name="robot_v3_gray">
-        <color rgba="0.82 0.82 0.82 1" />
-      </material>
-      <origin xyz="-0.41778609 -0.261 -0.24504893" rpy="1.5707963 -1.3089969 -3.1415927" />
-      <geometry>
-        <mesh filename="package://robot_description/meshes/robot_v3/part_022_solid_022.stl" scale="0.001 0.001 0.001" />
-      </geometry>
-    </visual>
-    <collision>
-      <origin xyz="-0.41778609 -0.261 -0.24504893" rpy="1.5707963 -1.3089969 -3.1415927" />
-      <geometry>
-        <mesh filename="package://robot_description/meshes/robot_v3/part_022_solid_022.stl" scale="0.001 0.001 0.001" />
-      </geometry>
-    </collision>
-  </link>
-  <link name="left_joint2">
-    <inertial>
-      <origin xyz="0.16099658 -2.2293885e-08 0.040000129" rpy="0 0 0" />
-      <mass value="4.3865155" />
-      <inertia ixx="0.015567363" iyy="0.01725914" izz="0.023316504" ixy="-9.380831e-09" ixz="5.7416863e-08" iyz="1.0365956e-08" />
-    </inertial>
-    <visual>
-      <material name="robot_v3_gray">
-        <color rgba="0.82 0.82 0.82 1" />
-      </material>
-      <origin xyz="-0.37224893 -0.261 0.45778609" rpy="-1.5707963 -0.26179939 0" />
-      <geometry>
-        <mesh filename="package://robot_description/meshes/robot_v3/part_023_solid_023.stl" scale="0.001 0.001 0.001" />
-      </geometry>
-    </visual>
-    <collision>
-      <origin xyz="-0.37224893 -0.261 0.45778609" rpy="-1.5707963 -0.26179939 0" />
-      <geometry>
-        <mesh filename="package://robot_description/meshes/robot_v3/part_023_solid_023.stl" scale="0.001 0.001 0.001" />
-      </geometry>
-    </collision>
-  </link>
-  <link name="left_joint3">
-    <inertial>
-      <origin xyz="-5.4838854e-08 2.313556e-09 0.23006341" rpy="0 0 0" />
-      <mass value="3.6348934" />
-      <inertia ixx="0.039501203" iyy="0.037988449" izz="0.011543295" ixy="-3.4108404e-10" ixz="-1.1585164e-08" iyz="2.5623177e-09" />
-    </inertial>
-    <visual>
-      <material name="robot_v3_gray">
-        <color rgba="0.82 0.82 0.82 1" />
-      </material>
-      <origin xyz="-0.41778609 -0.261 -0.55174893" rpy="1.5707963 -1.3089969 -3.1415927" />
-      <geometry>
-        <mesh filename="package://robot_description/meshes/robot_v3/part_024_solid_024.stl" scale="0.001 0.001 0.001" />
-      </geometry>
-    </visual>
-    <collision>
-      <origin xyz="-0.41778609 -0.261 -0.55174893" rpy="1.5707963 -1.3089969 -3.1415927" />
-      <geometry>
-        <mesh filename="package://robot_description/meshes/robot_v3/part_024_solid_024.stl" scale="0.001 0.001 0.001" />
-      </geometry>
-    </collision>
-  </link>
-  <link name="left_joint4">
-    <inertial>
-      <origin xyz="0.12628065 0.033836794 -0.069995268" rpy="0 0 0" />
-      <mass value="3.5816417" />
-      <inertia ixx="0.016515852" iyy="0.034995691" izz="0.029719472" ixy="-0.0053346689" ixz="2.2645394e-06" iyz="6.0678773e-07" />
-    </inertial>
-    <visual>
-      <material name="robot_v3_gray">
-        <color rgba="0.82 0.82 0.82 1" />
-      </material>
-      <origin xyz="-0.74019233 -0.63085793 -0.331" rpy="0 0 0" />
-      <geometry>
-        <mesh filename="package://robot_description/meshes/robot_v3/part_025_solid_025.stl" scale="0.001 0.001 0.001" />
-      </geometry>
-    </visual>
-    <collision>
-      <origin xyz="-0.74019233 -0.63085793 -0.331" rpy="0 0 0" />
-      <geometry>
-        <mesh filename="package://robot_description/meshes/robot_v3/part_025_solid_025.stl" scale="0.001 0.001 0.001" />
-      </geometry>
-    </collision>
-  </link>
-  <link name="left_joint5">
-    <inertial>
-      <origin xyz="-0.026243459 4.4018521e-10 0.128786" rpy="0 0 0" />
-      <mass value="2.5639763" />
-      <inertia ixx="0.013271127" iyy="0.01688134" izz="0.0092196052" ixy="-1.2416647e-10" ixz="-0.00039269081" iyz="7.1908348e-11" />
-    </inertial>
-    <visual>
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