Commit message: feat(rt-control): consume mapped arm inertia priors [ELECTRI-136]

File: src/description/robot_description/urdf/robot.urdf (robot description, URDF)
Before this commit: robot alfa_robot_v3, 36 links, 35 joints
Links:
- link left_link1: mass 3.4800785 -> 11.831
- link left_link2: mass 4.2029403 -> 8.774
- link left_link3: mass 3.6348934 -> 9.328
- link left_link4: mass 3.5816422 -> 3.715
- link left_link5: mass 2.5714853 -> 3.025
- link left_link6: mass 0.4671032 -> 1.505
- link right_link1: mass 3.4800784 -> 11.831
- link right_link2: mass 4.20294 -> 8.774
- link right_link3: mass 3.6348933 -> 9.328
- link right_link4: mass 3.5816414 -> 3.715
- link right_link5: mass 2.5714852 -> 3.025
- link right_link6: mass 0.4671031 -> 1.505

File: src/description/robot_description/urdf/robot_v3_1_1.xacro (robot description, xacro)
@@ -296,7 +296,7 @@
   <link name="right_link1">
     <inertial>
-      <origin xyz="0.026713078 -0.00035041598 0.12770383" rpy="0 0 0" />
-      <mass value="3.4800784" />
-      <inertia ixx="0.019990671" iyy="0.023084514" izz="0.018380907" ixy="-1.7698217e-05" ixz="-0.00075603007" iyz="-8.1890443e-05" />
+      <origin xyz="-0.017588 -0.0028841869 0.13899443" rpy="0 0 0" />
+      <mass value="11.831" />
+      <inertia ixx="0.049622545" ixy="-5.5706526e-06" ixz="-0.0031526704" iyy="0.049222113" iyz="0.0026718216" izz="0.041085115" />
     </inertial>
     <visual>
@@ -315,7 +315,7 @@
   <link name="right_link2">
     <inertial>
-      <origin xyz="-0.16472334 -1.1230144e-08 -0.040000126" rpy="0 0 0" />
-      <mass value="4.20294" />
-      <inertia ixx="0.014698616" iyy="0.015742815" izz="0.021103613" ixy="6.0405033e-09" ixz="5.5773205e-08" iyz="2.0954468e-08" />
+      <origin xyz="-0.167645195636 -0.00290158915044 -0.0417759956786" rpy="0 0 0" />
+      <mass value="8.774" />
+      <inertia ixx="0.0311528402451" ixy="-0.00337812479724" ixz="4.05105107462e-05" iyy="0.0350480907565" iyz="1.39633504305e-07" izz="0.0455440069984" />
     </inertial>
     <visual>
@@ -334,7 +334,7 @@
   <link name="right_link3">
     <inertial>
-      <origin xyz="-5.896457e-08 9.5061022e-10 0.23006341" rpy="0 0 0" />
-      <mass value="3.6348933" />
-      <inertia ixx="0.039501207" iyy="0.037988453" izz="0.011543294" ixy="-2.7986338e-10" ixz="-1.0220005e-08" iyz="2.5352711e-09" />
+      <origin xyz="-0.00177799026151 -0.00830873966354 0.299478137669" rpy="0 0 0" />
+      <mass value="9.328" />
+      <inertia ixx="0.0664349040005" ixy="-7.18247350348e-06" ixz="1.34258561537e-05" iyy="0.0559168058639" iyz="0.0154378537538" izz="0.0354338421355" />
     </inertial>
     <visual>
@@ -353,7 +353,7 @@
   <link name="right_link4">
     <inertial>
-      <origin xyz="-0.12628065 0.0338368 0.067995266" rpy="0 0 0" />
-      <mass value="3.5816414" />
-      <inertia ixx="0.016515852" iyy="0.034995692" izz="0.029719473" ixy="0.0053346708" ixz="2.262619e-06" iyz="-6.0604321e-07" />
+      <origin xyz="-0.181710062345 0.0468514706251 0.0728786181664" rpy="0 0 0" />
+      <mass value="3.715" />
+      <inertia ixx="0.0106536119821" ixy="0.00159006587363" ixz="0.00121891107665" iyy="0.016163942196" iyz="-0.000327481683669" izz="0.0128594488219" />
     </inertial>
     <visual>
@@ -372,7 +372,7 @@
   <link name="right_link5">
     <inertial>
-      <origin xyz="-0.026166805 0 0.12943329" rpy="0 0 0" />
-      <mass value="2.5714852" />
-      <inertia ixx="0.0133841" iyy="0.016999468" izz="0.0092322376" ixy="-4.8880228e-11" ixz="-0.00036895645" iyz="-3.280144e-11" />
+      <origin xyz="-0.00364697519152 0.0163528656786 0.108347889973" rpy="0 0 0" />
+      <mass value="3.025" />
+      <inertia ixx="0.0124624899837" ixy="-0.00029829186244" ixz="-7.54682908791e-06" iyy="0.0093224910792" iyz="0.00108600344158" izz="0.00722903693708" />
     </inertial>
     <visual>
@@ -391,7 +391,7 @@
   <link name="right_link6">
     <inertial>
-      <origin xyz="-0.05437806 0 -0.061500007" rpy="0 0 0" />
-      <mass value="0.4671031" />
-      <inertia ixx="0.00042456776" iyy="0.00052425348" izz="0.00053281307" ixy="1.7956352e-12" ixz="-9.302396e-11" iyz="2.7467158e-12" />
+      <origin xyz="-0.00211651236386 0.0112467822576 -0.0631829715852" rpy="0 0 0" />
+      <mass value="1.505" />
+      <inertia ixx="0.00224282643631" ixy="0.00072820819623" ixz="-2.35331962945e-08" iyy="0.00163958356386" iyz="-3.22712676169e-06" izz="0.00278854399983" />
     </inertial>
     <visual>
@@ -411,7 +411,7 @@
   <link name="left_link1">
     <inertial>
-      <origin xyz="0.026713079 -0.00035041871 0.12770383" rpy="0 0 0" />
-      <mass value="3.4800785" />
-      <inertia ixx="0.019990672" iyy="0.023084515" izz="0.018380907" ixy="-1.7697964e-05" ixz="-0.00075602927" iyz="-8.1890411e-05" />
+      <origin xyz="-0.017588 0.002883761 0.13899444" rpy="0 0 0" />
+      <mass value="11.831" />
+      <inertia ixx="0.049622545" ixy="5.5803149e-06" ixz="-0.0031526704" iyy="0.049222129" iyz="-0.0026717967" izz="0.041085099" />
     </inertial>
     <visual>
@@ -430,7 +430,7 @@
   <link name="left_link2">
     <inertial>
-      <origin xyz="0.16472335 1.2730856e-08 -0.040000127" rpy="0 0 0" />
-      <mass value="4.2029403" />
-      <inertia ixx="0.014698617" iyy="0.015742817" izz="0.021103615" ixy="5.4991019e-09" ixz="-5.5614112e-08" iyz="-2.0916153e-08" />
+      <origin xyz="0.167645195648 -0.00290158721144 -0.0417759956578" rpy="0 0 0" />
+      <mass value="8.774" />
+      <inertia ixx="0.0311528402451" ixy="0.00337812479694" ixz="-4.05105349997e-05" iyy="0.0350480907565" iyz="1.39708860644e-07" izz="0.0455440069984" />
     </inertial>
     <visual>
@@ -449,7 +449,7 @@
   <link name="left_link3">
     <inertial>
-      <origin xyz="-5.9080015e-08 2.5764869e-09 0.23006341" rpy="0 0 0" />
-      <mass value="3.6348934" />
-      <inertia ixx="0.039501204" iyy="0.03798845" izz="0.011543294" ixy="-3.3853139e-10" ixz="-9.1325076e-09" iyz="2.5994844e-09" />
+      <origin xyz="-0.00177799020186 0.00830876013458 0.299478136897" rpy="0 0 0" />
+      <mass value="9.328" />
+      <inertia ixx="0.0664349040006" ixy="7.18239909979e-06" ixz="1.34257447215e-05" iyy="0.0559168033067" iyz="-0.0154378554503" izz="0.0354338446927" />
     </inertial>
     <visual>
@@ -468,7 +468,7 @@
   <link name="left_link4">
     <inertial>
-      <origin xyz="0.12628066 0.033836802 0.068004734" rpy="0 0 0" />
-      <mass value="3.5816422" />
-      <inertia ixx="0.016515855" iyy="0.034995701" izz="0.029719482" ixy="-0.0053346723" ixz="2.2629901e-06" iyz="6.0627704e-07" />
+      <origin xyz="0.181710062738 0.0468514672726 0.0728786563338" rpy="0 0 0" />
+      <mass value="3.715" />
+      <inertia ixx="0.0106536121523" ixy="-0.00159006577844" ixz="-0.00121891132505" iyy="0.0161639422349" iyz="-0.000327481598673" izz="0.0128594486128" />
     </inertial>
     <visual>
@@ -487,7 +487,7 @@
   <link name="left_link5">
     <inertial>
-      <origin xyz="-0.026166799 2.9314955e-10 0.12943328" rpy="0 0 0" />
-      <mass value="2.5714853" />
-      <inertia ixx="0.013384094" iyy="0.016999459" izz="0.0092322348" ixy="-4.7934427e-12" ixz="-0.0003689586" iyz="-4.3290592e-11" />
+      <origin xyz="-0.00364697188213 -0.0163528148963 0.108347891438" rpy="0 0 0" />
+      <mass value="3.025" />
+      <inertia ixx="0.0124624899595" ixy="0.000298291926801" ixz="-7.5470916476e-06" iyy="0.00932249092272" iyz="-0.00108600363124" izz="0.00722903711778" />
     </inertial>
     <visual>
@@ -506,7 +506,7 @@
   <link name="left_link6">
     <inertial>
-      <origin xyz="0.054378045 -1.1235669e-09 -0.061499998" rpy="0 0 0" />
-      <mass value="0.4671032" />
-      <inertia ixx="0.00042456777" iyy="0.00052425357" izz="0.00053281318" ixy="2.0503291e-13" ixz="-1.1611109e-10" iyz="-2.6960516e-12" />
+      <origin xyz="0.00211651330106 0.0112467231276 -0.0631829607152" rpy="0 0 0" />
+      <mass value="1.505" />
+      <inertia ixx="0.00224282631569" ixy="-0.00072820824602" ixz="2.34413197691e-08" iyy="0.00163958368504" iyz="-3.22726418608e-06" izz="0.00278854399928" />
     </inertial>
     <visual>

File: src/description/robot_description/urdf/robot_v3_end_effectors.xacro (robot description, xacro)
@@ -3,8 +3,32 @@
   <xacro:macro name="v3_gripper" params="side">
     <link name="${side}_link7">
+      <xacro:if value="${side == 'left'}">
+      <xacro:property name="fixed_mass" value="4.968" />
+      <xacro:property name="fixed_cx" value="0.00791768934263" />
+      <xacro:property name="fixed_cy" value="0.0540799104769" />
+      <xacro:property name="fixed_cz" value="0.0701258437238" />
+      <xacro:property name="fixed_ixx" value="0.0279908997017" />
+      <xacro:property name="fixed_ixy" value="0.00130496404675" />
+      <xacro:property name="fixed_ixz" value="-3.28935086884e-05" />
+      <xacro:property name="fixed_iyy" value="0.022648579088" />
+      <xacro:property name="fixed_iyz" value="0.00613871307241" />
+      <xacro:property name="fixed_izz" value="0.0190359642103" />
+      </xacro:if>
+      <xacro:unless value="${side == 'left'}">
+      <xacro:property name="fixed_mass" value="4.968" />
+      <xacro:property name="fixed_cx" value="0.00791767509113" />
+      <xacro:property name="fixed_cy" value="-0.0540798334135" />
+      <xacro:property name="fixed_cz" value="0.0701258512213" />
+      <xacro:property name="fixed_ixx" value="0.0279908999288" />
+      <xacro:property name="fixed_ixy" value="-0.0013049632645" />
+      <xacro:property name="fixed_ixz" value="-3.28923344296e-05" />
+      <xacro:property name="fixed_iyy" value="0.0226485772779" />
+      <xacro:property name="fixed_iyz" value="-0.00613871361202" />
+      <xacro:property name="fixed_izz" value="0.0190359657934" />
+      </xacro:unless>
       <inertial>
-        <origin xyz="-0.007153 0.051039 0.078079" rpy="0 0 0" />
-        <mass value="4.750" />
-        <inertia ixx="0.023047048" ixy="0.001195672" ixz="0.000201380" iyy="0.013186943" iyz="-0.004207234" izz="0.024017065" />
+        <origin xyz="${fixed_cx} ${fixed_cy} ${fixed_cz}" rpy="0 0 0" />
+        <mass value="${fixed_mass}" />
+        <inertia ixx="${fixed_ixx}" ixy="${fixed_ixy}" ixz="${fixed_ixz}" iyy="${fixed_iyy}" iyz="${fixed_iyz}" izz="${fixed_izz}" />
       </inertial>
       <visual>
@@ -25,8 +49,32 @@
     </link>
     <link name="${side}_moving_jaw">
+      <xacro:if value="${side == 'left'}">
+      <xacro:property name="jaw_mass" value="0.086" />
+      <xacro:property name="jaw_cx" value="0.0312110612538" />
+      <xacro:property name="jaw_cy" value="-0.0474096878043" />
+      <xacro:property name="jaw_cz" value="0.109610525425" />
+      <xacro:property name="jaw_ixx" value="0.000118896982982" />
+      <xacro:property name="jaw_ixy" value="3.07524146586e-05" />
+      <xacro:property name="jaw_ixz" value="-6.87716451222e-05" />
+      <xacro:property name="jaw_iyy" value="0.000351487783728" />
+      <xacro:property name="jaw_iyz" value="-1.33502439253e-05" />
+      <xacro:property name="jaw_izz" value="0.00031015323329" />
+      </xacro:if>
+      <xacro:unless value="${side == 'left'}">
+      <xacro:property name="jaw_mass" value="0.086" />
+      <xacro:property name="jaw_cx" value="0.0312110359947" />
+      <xacro:property name="jaw_cy" value="0.0474097719652" />
+      <xacro:property name="jaw_cz" value="0.109610521055" />
+      <xacro:property name="jaw_ixx" value="0.00011889699562" />
+      <xacro:property name="jaw_ixy" value="-3.07524441807e-05" />
+      <xacro:property name="jaw_ixz" value="-6.87716525407e-05" />
+      <xacro:property name="jaw_iyy" value="0.000351487781911" />
+      <xacro:property name="jaw_iyz" value="1.33502310459e-05" />
+      <xacro:property name="jaw_izz" value="0.000310153222468" />
+      </xacro:unless>
       <inertial>
-        <origin xyz="-0.021670 0.021614 0.107390" rpy="0 0 0" />
-        <mass value="0.342" />
-        <inertia ixx="0.000402893" ixy="0.000112258" ixz="-0.000147231" iyy="0.001185610" iyz="-0.000064995" izz="0.001057162" />
+        <origin xyz="${jaw_cx} ${jaw_cy} ${jaw_cz}" rpy="0 0 0" />
+        <mass value="${jaw_mass}" />
+        <inertia ixx="${jaw_ixx}" ixy="${jaw_ixy}" ixz="${jaw_ixz}" iyy="${jaw_iyy}" iyz="${jaw_iyz}" izz="${jaw_izz}" />
       </inertial>
       <visual>
