Commit message: fix(rt-control): 台架方向全部 +1，改锁 robot_description 左 J3/J6 轴取反版本 [ELECTRI-127]

File: src/description/robot_description/urdf/robot_alfav3_mobile.urdf (robot description, URDF)
Before this commit: robot alfa_robot_v3, 32 links, 31 joints
Joints:
- joint left_joint3: axis 0 0 -1 -> 0 0 1
- joint left_joint6: axis 0 0 1 -> 0 0 -1

Commit message: chore(bench): 台架 ar@192.168.100.40 工作区现场快照 [arch-bench-field-20261030]
原样记录台架 ~/rt-control-electri127/robot_driver 在 6401efe 之上的全部未提交改动
（2026-10-30 导出），1361 个受跟踪文件与台架逐字节一致（SHA-256 清单比对），
仅排除 __pycache__/*.pyc。用于追溯与集成，不直接合并。

主要内容：
- bench_dual_arm / bench_right_arm 物理配置与各自的 stationary_enable、运动 scope；
- src/description/robot_description 为独立 robot_description 仓库
  feature/bilateral-j2-limits@c2b1ec5 的内容（逐文件一致）；
- rt_control_arm_console、真空网页、DPI 序列等现场功能及其记录。

File: src/description/robot_description/urdf/robot_alfav3_mobile.urdf (robot description, URDF)
Before this commit: robot alfa_robot_v3, 32 links, 31 joints
Links:
- removed link head
- removed link head_yaw
- added link H1_Link, mass 0.279891410655859; collision mesh filename=package://robot_description/mesh/head/H1_Link.STL; visual mesh filename=package://robot_description/mesh/head/H1_Link.STL
- added link H2_Link, mass 1.51565299644841; collision mesh filename=package://robot_description/mesh/head/H2_Link.STL; visual mesh filename=package://robot_description/mesh/head/H2_Link.STL
- added link Leye_link; visual mesh filename=package://robot_description/mesh/head/Leye_link.STL
- added link Reye_Link; visual mesh filename=package://robot_description/mesh/head/Reye_Link.STL
- added link mid360_Link, mass 0.375; collision mesh filename=package://robot_description/mesh/head/mid360_Link.STL; visual mesh filename=package://robot_description/mesh/head/mid360_Link.STL
- link arm_carriage: mass 42.349928 -> 43.0078185286443; geometry collision mesh filename=package://robot_description/mesh/torso/base_link.STL; visual mesh filename=package://robot_description/mesh/torso/base_link.STL
- link base_link: geometry collision mesh filename=package://robot_description/mesh/chassis/part_001_solid_001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 scale=0.001 0.001 0.001; collision mesh filename=package://robot_description/mesh/chassis/part_048_solid_048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 scale=0.001 0.001 0.001
- link left_link1: geometry collision mesh filename=package://robot_description/mesh/arms/collision/left_link1.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; visual mesh filename=package://robot_description/mesh/arms/visual/left_link1.STL
- link left_link2: geometry collision mesh filename=package://robot_description/mesh/arms/collision/left_link2.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; visual mesh filename=package://robot_description/mesh/arms/visual/left_link2.STL
- link left_link3: geometry collision mesh filename=package://robot_description/mesh/arms/collision/left_link3.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; visual mesh filename=package://robot_description/mesh/arms/visual/left_link3.STL
- link left_link4: geometry collision mesh filename=package://robot_description/mesh/arms/collision/left_link4.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; visual mesh filename=package://robot_description/mesh/arms/visual/left_link4.STL
- link left_link5: geometry collision mesh filename=package://robot_description/mesh/arms/collision/left_link5.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; visual mesh filename=package://robot_description/mesh/arms/visual/left_link5.STL
- link left_link6: geometry collision mesh filename=package://robot_description/mesh/arms/collision/left_link6.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; visual mesh filename=package://robot_description/mesh/arms/visual/left_link6.STL
- link left_link7: geometry collision mesh filename=package://robot_description/mesh/arms/collision/left_link7.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; visual mesh filename=package://robot_description/mesh/arms/visual/left_link7.STL
- link left_tool_link: geometry collision mesh filename=package://robot_description/mesh/arms/collision/left_tool_l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; visual mesh filename=package://robot_description/mesh/arms/visual/left_tool_link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
- link right_link1: geometry collision mesh filename=package://robot_description/mesh/arms/collision/right_link1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; visual mesh filename=package://robot_description/mesh/arms/visual/right_link1.STL
- link right_link2: geometry collision mesh filename=package://robot_description/mesh/arms/collision/right_link2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; visual mesh filename=package://robot_description/mesh/arms/visual/right_link2.STL
- link right_link3: geometry collision mesh filename=package://robot_description/mesh/arms/collision/right_link3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; visual mesh filename=package://robot_description/mesh/arms/visual/right_link3.STL
- link right_link4: geometry collision mesh filename=package://robot_description/mesh/arms/collision/right_link4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; visual mesh filename=package://robot_description/mesh/arms/visual/right_link4.STL
- link right_link5: geometry collision mesh filename=package://robot_description/mesh/arms/collision/right_link5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; visual mesh filename=package://robot_description/mesh/arms/visual/right_link5.STL
- link right_link6: geometry collision mesh filename=package://robot_description/mesh/arms/collision/right_link6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; visual mesh filename=package://robot_description/mesh/arms/visual/right_link6.STL
- link right_link7: geometry collision mesh filename=package://robot_description/mesh/arms/collision/right_link7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; visual mesh filename=package://robot_description/mesh/arms/visual/right_link7.STL
- link right_tool_link: geometry collision mesh filename=package://robot_description/mesh/arms/collision/right_tool_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; visual mesh filename=package://robot_description/mesh/arms/visual/right_tool_lin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
- link steer1: geometry collision mesh filename=package://robot_description/mesh/chassis/part_061_solid_061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 scale=0.001 0.001 0.001; visual mesh filename=package://robot_description/mesh/chassis/part_061_solid_061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 scale=0.001 0.001 0.001
- link steer2: geometry collision mesh filename=package://robot_description/mesh/chassis/part_059_solid_059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 scale=0.001 0.001 0.001; visual mesh filename=package://robot_description/mesh/chassis/part_059_solid_059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 scale=0.001 0.001 0.001
- link steer3: geometry collision mesh filename=package://robot_description/mesh/chassis/part_065_solid_065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 scale=0.001 0.001 0.001; visual mesh filename=package://robot_description/mesh/chassis/part_065_solid_065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 scale=0.001 0.001 0.001
- link steer4: geometry collision mesh filename=package://robot_description/mesh/chassis/part_063_solid_063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 scale=0.001 0.001 0.001; visual mesh filename=package://robot_description/mesh/chassis/part_063_solid_063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 scale=0.001 0.001 0.001
- link wheel1: geometry collision mesh filename=package://robot_description/mesh/chassis/part_062_solid_062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 scale=0.001 0.001 0.001; visual mesh filename=package://robot_description/mesh/chassis/part_062_solid_062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 scale=0.001 0.001 0.001
- link wheel2: geometry collision mesh filename=package://robot_description/mesh/chassis/part_060_solid_060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 scale=0.001 0.001 0.001; visual mesh filename=package://robot_description/mesh/chassis/part_060_solid_060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 scale=0.001 0.001 0.001
- link wheel3: geometry collision mesh filename=package://robot_description/mesh/chassis/part_066_solid_066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 scale=0.001 0.001 0.001; visual mesh filename=package://robot_description/mesh/chassis/part_066_solid_066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 scale=0.001 0.001 0.001
- link wheel4: geometry collision mesh filename=package://robot_description/mesh/chassis/part_064_solid_064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 scale=0.001 0.001 0.001; visual mesh filename=package://robot_description/mesh/chassis/part_064_solid_064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 scale=0.001 0.001 0.001
Joints:
- removed joint head_joint
- removed joint head_pitch_joint
- added joint H1_joint: type revolute, parent arm_carriage, child H1_Link, origin xyz=0.26699999999999902 0 0.36514999999999997 rpy=3.1415926535897931 0 0, axis 0 0 1, limit lower=-3.141592653589793 upper=3.141592653589793 effort=10 velocity=5
- added joint H2_joint: type revolute, parent H1_Link, child H2_Link, origin xyz=0 0 0.24625009252407 rpy=1.5707963267949 0 0, axis 0 0 1, limit lower=-3.141592653589793 upper=3.141592653589793 effort=10 velocity=5
- added joint Leye_joint: type fixed, parent H2_Link, child Leye_link, origin xyz=0.012866 0.11171 -0.06 rpy=-1.5708 0 0, axis 0 0 0
- added joint Reye_joint: type fixed, parent H2_Link, child Reye_Link, origin xyz=0.012866 0.11171 0.06 rpy=-1.5708 0 0, axis 0 0 0
- added joint mid360_joint: type fixed, parent H2_Link, child mid360_Link, origin xyz=0.03857 0.066019 0 rpy=-1.5708 0 -0.37885, axis 0 0 0
- joint left_joint1: limit lower=-3.141592653589793 upper=3.141592653589793 effort=647 velocity=1.309 -> lower=-2.792526803190927 upper=2.792526803190927 effort=647 velocity=1.3089969389957472
- joint left_joint2: limit lower=-1.8325957145940461 upper=1.8325957145940461 effort=647 velocity=1.309 -> lower=-1.6057029118347832 upper=2.129301687433082 effort=647 velocity=1.3089969389957472
- joint left_joint3: limit lower=-3.141592653589793 upper=3.141592653589793 effort=484 velocity=1.309 -> lower=-2.792526803190927 upper=2.792526803190927 effort=484 velocity=1.3089969389957472
- joint left_joint4: limit lower=-2.530727415391778 upper=2.530727415391778 effort=459 velocity=1.749 -> lower=-2.6179938779914944 upper=2.6179938779914944 effort=459 velocity=1.7488199104983182
- joint left_joint5: limit lower=-3.141592653589793 upper=3.141592653589793 effort=217 velocity=2.618 -> lower=-2.792526803190927 upper=2.792526803190927 effort=204 velocity=3.1415926535897927; origin xyz=0 0.474 0 rpy=-1.5707963267949 0 0 -> xyz=0 0.474 0 rpy=-1.5707963267949 3.141592653589793 0
- joint left_joint6: limit lower=-1.9198621771937625 upper=1.9198621771937625 effort=107 velocity=3.142 -> lower=-2.356194490192345 upper=2.356194490192345 effort=107 velocity=3.1415926535897927
- joint left_joint7: limit lower=-3.141592653589793 upper=3.141592653589793 effort=36 velocity=3.142 -> lower=-2.792526803190927 upper=2.792526803190927 effort=36 velocity=3.1415926535897927
- joint right_joint1: limit lower=-3.141592653589793 upper=3.141592653589793 effort=647 velocity=1.309 -> lower=-2.792526803190927 upper=2.792526803190927 effort=647 velocity=1.3089969389957472
- joint right_joint2: limit lower=-1.8325957145940461 upper=1.8325957145940461 effort=647 velocity=1.309 -> lower=-1.6057029118347832 upper=2.129301687433082 effort=647 velocity=1.3089969389957472
- joint right_joint3: axis 0 0 -1 -> 0 0 1; limit lower=-3.141592653589793 upper=3.141592653589793 effort=484 velocity=1.309 -> lower=-2.792526803190927 upper=2.792526803190927 effort=484 velocity=1.3089969389957472
- joint right_joint4: axis 0 0 -1 -> 0 0 1; limit lower=-2.530727415391778 upper=2.530727415391778 effort=459 velocity=1.749 -> lower=-2.6179938779914944 upper=2.6179938779914944 effort=459 velocity=1.7488199104983182
- joint right_joint5: limit lower=-3.141592653589793 upper=3.141592653589793 effort=217 velocity=2.618 -> lower=-2.792526803190927 upper=2.792526803190927 effort=204 velocity=3.1415926535897927; origin xyz=0 -0.474000000000003 0 rpy=1.5707963267949 0 0 -> xyz=0 -0.474000000000003 0 rpy=-1.570796326795 3.14159265359 3.14159265359
- joint right_joint6: limit lower=-1.9198621771937625 upper=1.9198621771937625 effort=107 velocity=3.142 -> lower=-2.356194490192345 upper=2.356194490192345 effort=107 velocity=3.1415926535897927
- joint right_joint7: limit lower=-3.141592653589793 upper=3.141592653589793 effort=36 velocity=3.142 -> lower=-2.792526803190927 upper=2.792526803190927 effort=36 velocity=3.1415926535897927
