Commit message: feat(rt-control): 迁入研华底盘台架已验证事实与 BRT EDS [ELECTRI-127]
- 八轴环位、方向、计数、零点，四编码器节点/方向/偏置/分辨率/圈数，
  模块坐标与轮径写入机型、单机与设备数据；轮组键改为 module_1..4。
- Kinco profile 填入身份、DC、看门狗、反馈超时、停稳阈值与模式确认超时；
  组件速度上限按转向/行走分开。
- 渲染器导出 steering_to_yaw_sign 与 encoder_revolutions 并绑定到控制器/传感器。
- 控制器策略按用户值设置速度与加速度（轮面 m/s、m/s²），协方差为占位值。
- 迁入 BRT EDS 厂家原件与兼容文件及测试。

File: src/rt_control/rt_control_machine_config/machines/Alfa_V3/chassis.mock.urdf (robot description, URDF)
Before this commit: robot swerve_mock, 9 links, 8 joints
Links:
- removed link d0_link
- removed link d1_link
- removed link d2_link
- removed link d3_link
- removed link s0_link
- removed link s1_link
- removed link s2_link
- removed link s3_link
- added link steer1
- added link steer2
- added link steer3
- added link steer4
- added link wheel1
- added link wheel2
- added link wheel3
- added link wheel4
Joints:
- removed joint d0
- removed joint d1
- removed joint d2
- removed joint d3
- removed joint s0
- removed joint s1
- removed joint s2
- removed joint s3
- added joint steer1_joint: type continuous, parent base, child steer1, axis 0 0 1
- added joint steer2_joint: type continuous, parent base, child steer2, axis 0 0 1
- added joint steer3_joint: type continuous, parent base, child steer3, axis 0 0 1
- added joint steer4_joint: type continuous, parent base, child steer4, axis 0 0 1
- added joint wheel1_joint: type continuous, parent base, child wheel1, axis 0 0 1
- added joint wheel2_joint: type continuous, parent base, child wheel2, axis 0 0 1
- added joint wheel3_joint: type continuous, parent base, child wheel3, axis 0 0 1
- added joint wheel4_joint: type continuous, parent base, child wheel4, axis 0 0 1
